Commit message: - UR10 com a garra exibido no Gazebo, controladores ok - UR10 com garra pacote no moveit parcialmente configurado (precisa ajustes para o moveit conseguir movimentar o robô no Gazebo)

File: catkin_ws/src/ur10_moveit_with_gripper_config/config/gazebo_ur10_with_gripper.urdf (robot description, URDF)
Before this commit: robot ur10_with_gripper, 16 links, 15 joints
Links:
- link pg70_base_link: mass 0.1 -> 0.5
- link pg70_finger_left_link: mass 0.1 -> 0.05
- link pg70_finger_right_link: mass 0.1 -> 0.05
- link pg70_fingertip_left_link: mass 0.1 -> 0.02
- link pg70_fingertip_right_link: mass 0.1 -> 0.02
Joints:
- joint pg70_finger_right_joint: origin xyz=0 0 0.0789 rpy=-0 0 0 -> xyz=0 0 0.0789 rpy=0 0 0

File: catkin_ws/src/ur10_with_gripper/urdf/ur10_with_gripper.urdf.xacro (robot description, xacro)
@@ -2,12 +2,21 @@
 <robot xmlns:xacro="http://www.ros.org/wiki/xacro" name="ur10_with_gripper">
   <!-- Inclui o UR10 -->
+  <!-- Definição do parâmetro para o tipo de interface de hardware -->
+  <xacro:property name="transmission_hw_interface" value="hardware_interface/EffortJointInterface"/>
   <xacro:include filename="$(find ur_description)/urdf/inc/ur10_macro.xacro"/>
-  <xacro:ur10_robot prefix="" />
-  <!-- Inclui a garra -->
+  <!-- Instancia o UR10 com o parâmetro -->
+  <xacro:ur10_robot
+    prefix=""
+    transmission_hw_interface="${transmission_hw_interface}" />
+  <!-- <xacro:ur10_robot prefix="" /> -->
   <!-- Inclui a garra PG70 -->
-    <xacro:include filename="$(find schunk_pg70)/urdf/pg70.urdf.xacro"/>
+    <xacro:include filename="$(find ur10_with_gripper)/urdf/pg70_with_control.urdf.xacro"/>
     <!-- Adiciona a garra ao final do braço -->
     <xacro:schunk_pg70 parent="tool0" name="pg70">
         <origin xyz="0 0 0" rpy="0 0 0"/>
     </xacro:schunk_pg70>
+  <!-- Plugin para ROS control via Gazebo -->
+  <gazebo>
+    <plugin name="gazebo_ros_control" filename="libgazebo_ros_control.so"/>
+  </gazebo>
 </robot>
